File: cyton hat/Daisy Functionality.kicad_sch (KiCad schematic)
At the start: 28 parts, among them U1 ADS129x

Commit message: finished layout
Parts:
- C10, C11, C14, C15, C6, C7, C8, C9: footprint (none) -> Capacitor_SMD:C_0402_1005Metric
- C12: footprint (none) -> Capacitor_SMD:C_1206_3216Metric
- C13: footprint (none) -> Capacitor_SMD:C_0603_1608Metric
- D1, D2, D3, D4, D5, D6: footprint DCK6_TEX -> TSV - Diodes:TPD4E1B06DCKR
- R6: footprint (none) -> Resistor_SMD:R_0402_1005Metric
Connections:
- net SRB1: no longer U1.17 (TESTP_PACE_OUT1)
- net _SRB1: now also U1.17 (TESTP_PACE_OUT1)
Changed lines of the file:
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@@
     (effects (font (size 1.27 1.27)) (justify left bottom))
   )
-  (label "SRB1" (at 447.675 206.375 0)
+  (label "_SRB1" (at 447.675 206.375 0)
     (effects (font (size 1.27 1.27)) (justify left bottom))
   )
@@
       (effects (font (size 1.524 1.524)))
     )
-    (property "Footprint" "DCK6_TEX" (id 2) (at 97.155 184.404 0)
+    (property "Footprint" "TSV - Diodes:TPD4E1B06DCKR" (id 2) (at 97.155 184.404 0)
       (effects (font (size 1.524 1.524)) hide)
     )
@@
       (effects (font (size 1.524 1.524)))
     )
-    (property "Footprint" "DCK6_TEX" (id 2) (at 101.6 336.804 0)
+    (property "Footprint" "TSV - Diodes:TPD4E1B06DCKR" (id 2) (at 101.6 336.804 0)
       (effects (font (size 1.524 1.524)) hide)
     )
@@
       (effects (font (size 1.27 1.27)) (justify left))
     )
-    (property "Footprint" "" (id 2) (at 375.6152 274.955 0)
+    (property "Footprint" "Capacitor_SMD:C_0402_1005Metric" (id 2) (at 375.6152 274.955 0)
       (effects (font (size 1.27 1.27)) hide)
     )
@@
       (effects (font (size 1.27 1.27)) (justify left))
     )
-    (property "Footprint" "" (id 2) (at 322.9102 248.92 0)
+    (property "Footprint" "Capacitor_SMD:C_0402_1005Metric" (id 2) (at 322.9102 248.92 0)
       (effects (font (size 1.27 1.27)) hide)
     )
@@
       (effects (font (size 1.27 1.27)) (justify left))
     )
-    (property "Footprint" "" (id 2) (at 343.8652 292.735 0)
+    (property "Footprint" "Capacitor_SMD:C_0402_1005Metric" (id 2) (at 343.8652 292.735 0)
       (effects (font (size 1.27 1.27)) hide)
     )
@@
       (effects (font (size 1.27 1.27)) (justify left))
     )
-    (property "Footprint" "" (id 2) (at 473.837 186.055 90)
+    (property "Footprint" "Resistor_SMD:R_0402_1005Metric" (id 2) (at 473.837 186.055 90)
       (effects (font (size 1.27 1.27)) hide)
     )
@@
       (effects (font (size 1.524 1.524)))
     )
-    (property "Footprint" "DCK6_TEX" (id 2) (at 111.76 47.244 0)
+    (property "Footprint" "TSV - Diodes:TPD4E1B06DCKR" (id 2) (at 111.76 47.244 0)
       (effects (font (size 1.524 1.524)) hide)
     )
@@
       (effects (font (size 1.524 1.524)))
     )
-    (property "Footprint" "DCK6_TEX" (id 2) (at 99.695 233.934 0)
+    (property "Footprint" "TSV - Diodes:TPD4E1B06DCKR" (id 2) (at 99.695 233.934 0)
       (effects (font (size 1.524 1.524)) hide)
     )
@@
       (effects (font (size 1.27 1.27)) (justify left))
     )
-    (property "Footprint" "" (id 2) (at 334.3402 292.735 0)
+    (property "Footprint" "Capacitor_SMD:C_0402_1005Metric" (id 2) (at 334.3402 292.735 0)
       (effects (font (size 1.27 1.27)) hide)
     )
@@
       (effects (font (size 1.27 1.27)) (justify left))
     )
-    (property "Footprint" "" (id 2) (at 362.2802 274.955 0)
+    (property "Footprint" "Capacitor_SMD:C_0603_1608Metric" (id 2) (at 362.2802 274.955 0)
       (effects (font (size 1.27 1.27)) hide)
     )
@@
       (effects (font (size 1.27 1.27)) (justify left))
     )
-    (property "Footprint" "" (id 2) (at 334.3402 248.92 0)
+    (property "Footprint" "Capacitor_SMD:C_0402_1005Metric" (id 2) (at 334.3402 248.92 0)
       (effects (font (size 1.27 1.27)) hide)
     )
@@
       (effects (font (size 1.27 1.27)) (justify left))
     )
-    (property "Footprint" "" (id 2) (at 357.2002 248.92 0)
+    (property "Footprint" "Capacitor_SMD:C_0402_1005Metric" (id 2) (at 357.2002 248.92 0)
       (effects (font (size 1.27 1.27)) hide)
     )
@@
       (effects (font (size 1.524 1.524)))
     )
-    (property "Footprint" "DCK6_TEX" (id 2) (at 100.965 286.004 0)
+    (property "Footprint" "TSV - Diodes:TPD4E1B06DCKR" (id 2) (at 100.965 286.004 0)
       (effects (font (size 1.524 1.524)) hide)
     )
@@
       (effects (font (size 1.524 1.524)))
     )
-    (property "Footprint" "DCK6_TEX" (id 2) (at 94.615 124.714 0)
+    (property "Footprint" "TSV - Diodes:TPD4E1B06DCKR" (id 2) (at 94.615 124.714 0)
       (effects (font (size 1.524 1.524)) hide)
     )
@@
       (effects (font (size 1.27 1.27)) (justify left))
     )
-    (property "Footprint" "" (id 2) (at 344.5002 248.92 0)
+    (property "Footprint" "Capacitor_SMD:C_0402_1005Metric" (id 2) (at 344.5002 248.92 0)
       (effects (font (size 1.27 1.27)) hide)
     )
@@
       (effects (font (size 1.27 1.27)) (justify left))
     )
-    (property "Footprint" "" (id 2) (at 463.8802 189.865 0)
+    (property "Footprint" "Capacitor_SMD:C_0402_1005Metric" (id 2) (at 463.8802 189.865 0)
       (effects (font (size 1.27 1.27)) hide)
     )
@@
       (effects (font (size 1.27 1.27)) (justify left))
     )
-    (property "Footprint" "" (id 2) (at 367.9952 248.92 0)
-      (effects (font (size 1.27 1.27)) hide)
-    )
+    (property "Footprint" "Capacitor_SMD:C_1206_3216Metric" (id 2) (at 367.9952 248.92 0)
+      (effects (font (size 1.27 1.27)) hide)
+    )
