File: cyton hat/USB Dongle.kicad_sch (KiCad schematic)
At the start: 19 parts, among them U2 CP2102N-Axx-xQFN24

Commit message: fixed D9 footprint problem
Parts:
- D9: footprint ESDALC6V1-1M2:ESDALC6V1-1M2 -> TSV - Diodes:ESDALC6V1-1M2
Changed lines of the file:
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@@
       (effects (font (size 1.27 1.27)) (justify left))
     )
-    (property "Footprint" "ESDALC6V1-1M2:ESDALC6V1-1M2" (id 2) (at 144.78 67.31 0)
+    (property "Footprint" "TSV - Diodes:ESDALC6V1-1M2" (id 2) (at 144.78 67.31 0)
       (effects (font (size 1.27 1.27)) hide)
     )
