File: hardware/cyton wired/Daisy Functionality.kicad_sch (KiCad schematic)
At the start: 30 parts, among them U1 ADS129x

Commit message: added power supply
Parts:
- C1: footprint Capacitor Arrays:CAPCAXE50P210X130X94-8N -> Capacitor_SMD:C_0402_1005Metric
Changed lines of the file:
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@@
       (effects (font (size 1.27 1.27)) (justify left bottom) hide)
     )
-    (property "Footprint" "Capacitor Arrays:CAPCAXE50P210X130X94-8N" (id 2) (at 181.61 356.87 0)
+    (property "Footprint" "Capacitor_SMD:C_0402_1005Metric" (id 2) (at 181.61 356.87 0)
       (effects (font (size 1.27 1.27)) (justify bottom) hide)
     )
@@
       (effects (font (size 1.27 1.27)) (justify left bottom) hide)
     )
-    (property "Footprint" "Capacitor Arrays:CAPCAXE50P210X130X94-8N" (id 2) (at 171.45 356.87 0)
+    (property "Footprint" "Capacitor_SMD:C_0402_1005Metric" (id 2) (at 171.45 356.87 0)
       (effects (font (size 1.27 1.27)) (justify bottom) hide)
     )
@@
       (effects (font (size 1.27 1.27)) (justify left bottom) hide)
     )
-    (property "Footprint" "Capacitor Arrays:CAPCAXE50P210X130X94-8N" (id 2) (at 161.29 356.87 0)
+    (property "Footprint" "Capacitor_SMD:C_0402_1005Metric" (id 2) (at 161.29 356.87 0)
       (effects (font (size 1.27 1.27)) (justify bottom) hide)
     )
@@
       (effects (font (size 1.27 1.27)) (justify left bottom) hide)
     )
-    (property "Footprint" "Capacitor Arrays:CAPCAXE50P210X130X94-8N" (id 2) (at 191.77 356.87 0)
-      (effects (font (size 1.27 1.27)) (justify bottom) hide)
-    )
+    (property "Footprint" "Capacitor_SMD:C_0402_1005Metric" (id 2) (at 191.77 356.87 0)
+      (effects (font (size 1.27 1.27)) (justify bottom) hide)
+    )

Commit message: added power supply
Parts:
- C1: footprint Capacitor_SMD:C_0402_1005Metric -> Capacitor Arrays:CAPCAXE50P210X130X94-8N
Changed lines of the file:
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@@
       (effects (font (size 1.27 1.27)) (justify left bottom) hide)
     )
-    (property "Footprint" "Capacitor_SMD:C_0402_1005Metric" (id 2) (at 181.61 356.87 0)
+    (property "Footprint" "Capacitor Arrays:CAPCAXE50P210X130X94-8N" (id 2) (at 181.61 356.87 0)
       (effects (font (size 1.27 1.27)) (justify bottom) hide)
     )
@@
       (effects (font (size 1.27 1.27)) (justify left bottom) hide)
     )
-    (property "Footprint" "Capacitor_SMD:C_0402_1005Metric" (id 2) (at 171.45 356.87 0)
+    (property "Footprint" "Capacitor Arrays:CAPCAXE50P210X130X94-8N" (id 2) (at 171.45 356.87 0)
       (effects (font (size 1.27 1.27)) (justify bottom) hide)
     )
@@
       (effects (font (size 1.27 1.27)) (justify left bottom) hide)
     )
-    (property "Footprint" "Capacitor_SMD:C_0402_1005Metric" (id 2) (at 161.29 356.87 0)
+    (property "Footprint" "Capacitor Arrays:CAPCAXE50P210X130X94-8N" (id 2) (at 161.29 356.87 0)
       (effects (font (size 1.27 1.27)) (justify bottom) hide)
     )
@@
       (effects (font (size 1.27 1.27)) (justify left bottom) hide)
     )
-    (property "Footprint" "Capacitor_SMD:C_0402_1005Metric" (id 2) (at 191.77 356.87 0)
-      (effects (font (size 1.27 1.27)) (justify bottom) hide)
-    )
+    (property "Footprint" "Capacitor Arrays:CAPCAXE50P210X130X94-8N" (id 2) (at 191.77 356.87 0)
+      (effects (font (size 1.27 1.27)) (justify bottom) hide)
+    )
