File: hardware/cyton wired/cyton wired.kicad_sch (KiCad schematic)
At the start: 13 parts, among them J1 Conn_02x13_Odd_Even, J2 Conn_01x08, J3 Conn_01x04, J4 Conn_01x02, J5 Conn_01x04

Commit message: snapshot of current MCU work
Connections:
- no-connect marks 8 -> 11
Other:
- added sheet MCU (MCU.kicad_sch)

Commit message: finished layout working on silkscreen
Connections:
- net GNDA: now also J3.4 (Pin_4)
- net VDD: now also J3.3 (Pin_3)
- net BOOT_EN: now reaches J5.1 (Pin_1)
- net MCLR: now reaches J5.2 (Pin_2)
- net D18: now reaches J5.3 (Pin_3)
- net PGD: now reaches J5.4 (Pin_4)
- net D13: now reaches J3.1 (Pin_1)
- net PGC: now reaches J3.2 (Pin_2)
- net _MISO renamed MISO
- no-connect marks 11 -> 3
Other:
- sheet Daisy Functionality: file Daisy Functionality.kicad_sch -> ../shared schematics/Daisy Functionality.kicad_sch
- sheet Daisy Functionality ports: added CS, DRDY, MISO; removed CS2, _MISO
- sheet MCU: file MCU.kicad_sch -> ../shared schematics/MCU.kicad_sch
- sheet MCU ports: added MCLR; removed none
- sheet Power Supply: file Power Supply.kicad_sch -> ../shared schematics/Power Supply.kicad_sch
- sheet USB Dongle: file USB Dongle.kicad_sch -> ../shared schematics/USB Dongle.kicad_sch
