File: hardware/shared schematics/ADS129X-X functionality.kicad_sch (KiCad schematic)
At the start: 30 parts, among them U1 ADS129x

Commit message: changed C27 from an 0402 package to a 0201 package
Parts:
- C27: footprint Capacitor_SMD:C_0201_0603Metric -> Capacitor_SMD:C_0402_1005Metric
