File: hardware/shared schematics/USB Dongle.kicad_sch (KiCad schematic)
At the start: 19 parts, among them U2 CP2102N-Axx-xQFN24

Commit message: changed C27 from an 0402 package to a 0201 package
Parts:
- C17, C18: footprint Capacitor_SMD:C_0201_0603Metric -> Capacitor_SMD:C_0402_1005Metric
Changed lines of the file:
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@@
       (effects (font (size 1.27 1.27)) (justify left))
     )
-    (property "Footprint" "Capacitor_SMD:C_0201_0603Metric" (at 134.3152 132.08 0)
+    (property "Footprint" "Capacitor_SMD:C_0402_1005Metric" (at 134.3152 132.08 0)
       (effects (font (size 1.27 1.27)) hide)
     )
@@
       (effects (font (size 1.27 1.27)) (justify left))
     )
-    (property "Footprint" "Capacitor_SMD:C_0201_0603Metric" (at 110.1852 132.08 0)
+    (property "Footprint" "Capacitor_SMD:C_0402_1005Metric" (at 110.1852 132.08 0)
       (effects (font (size 1.27 1.27)) hide)
     )
